File: TeamG_PCB.brd (EAGLE design)
At the start: 100 x 80 mm, 34 parts, among them U1 MIC29300-3.3WU, U2 MIC29300-5.0WU, U3 MIC29300-12WU

Commit message: Update
Parts:
- removed 12VLED, 3VLED, 5VLED: 0, led:1206
- removed C6: 1µF, rcl:C1210
- removed CPU_3P3V, ENCODER_5V, LIDAR_12V, MOTOR_24V, WIFI_5V: C-GRID-02-70543, con-molex:70543-02
- removed CR3: SMAJ26A-E3/61, SMAJ26A-E361:DIODE_DO-214AC
- removed R7: 65Ω, rcl:R1206
- removed R8: 150Ω, rcl:R1206
- added C4: 1µF, rcl:C1210
- added CPU, ENCODER, LIDAR, MOTOR, WIFI: C-GRID-02-70543, con-molex:70543-02
- added CR2: SMAJ26A-E3/61, SMAJ26A-E361:DIODE_DO-214AC
- added LED_12V, LED_3V, LED_5V: 0, led:1206
- added R2: 100Ω, rcl:R1206
- added R3: 150Ω, rcl:R1206
- D1, D2: value P4SMA16A -> VISHAY_SMBJ3V3-E3-52VISHAY_SMBJ3V3-E3-52_0_0; device P4SMA16A:DIOM4325X250N -> SMBJ3V3-E352:VISHAY_SMBJ3V3-E3-52_0
- D3, D4: value VISHAY_SMBJ3V3-E3-52VISHAY_SMBJ3V3-E3-52_0_0 -> SMAJ5.0; device SMBJ3V3-E352:VISHAY_SMBJ3V3-E3-52_0 -> SMAJ5.0:DIOM4325X250N
- D5, D6: value SMAJ5.0 -> P4SMA16A; device SMAJ5.0:DIOM4325X250N -> P4SMA16A:DIOM4325X250N
- F2: value 3A -> 1.5A
- F4: value 1.5A -> 3A
- R1: value 1100Ω -> 1000Ω
- moved U2 78.8 mm to (12.7, 36.8), turned to 90 degrees
- moved U3 77.4 mm to (40.6, 71.1), turned to 0 degrees
- moved D4 74.0 mm to (78.7, 53.3), turned to 90 degrees
- moved D6 68.3 mm to (77.5, 11.4), turned to 270 degrees
- moved D3 60.5 mm to (67.3, 50.8), turned to 180 degrees
- moved U1 52.1 mm to (48.3, 34.3), turned to 0 degrees
- moved D5 51.6 mm to (73.7, 24.1), turned to 90 degrees
- moved F3 48.5 mm to (35.6, 39.4), turned to 180 degrees
- moved D2 46.4 mm to (78.7, 40.6), turned to 90 degrees
- moved F5 37.4 mm to (45.7, 54.6), turned to 0 degrees
- moved D1 35.6 mm to (78.7, 31.8), turned to 90 degrees
- moved CR1 34.3 mm to (24.1, 67.3), turned to 90 degrees
- moved F1 28.5 mm to (15.2, 57.1)
- moved F2 26.2 mm to (62.2, 29.2), turned to 270 degrees
- moved C2 23.0 mm to (30.5, 24.1), turned to 180 degrees
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Connections:
- removed net 24V_SAFE: C1.1, CR1.1, CR3.1, F5.1, R1.2, U1.1, U2.1, U3.1
- removed net 5V_SAFE: C3.1, D5.C, D6.C, ENCODER_5V.1, R8.2, WIFI_5V.1
- removed net N$10: C2.1, CPU_3P3V.1, D3.1, D4.1, R7.2
- removed net N$12: C6.1, D1.C, D2.C, LIDAR_12V.1, R4.2
- removed net N$4 (its old number): D1.A, F2.1
- new net 12V: C4.1, D5.C, D6.C, LIDAR.1, R4.2
- new net 24V: C1.1, CR1.1, CR2.1, F5.1, R1.2, U1.1, U2.1, U3.1
- new net 3.3V: C2.1, CPU.1, D1.1, D2.1, R2.2
- new net 5V: C3.1, D3.C, D4.C, ENCODER.1, R3.2, WIFI.1
- new net N$15: D3.A, F3.1
- net GND: now also 24V.2, C4.2, CPU.2, CR2.2, D2.2, D4.A, ENCODER.2, LED_12V.C, LED_3V.C, LED_5V.C, LIDAR.2, MOTOR.2, WIFI.2; no longer 12VLED.C, 24V.1, 3VLED.C, 5VLED.C, C6.2, CPU_3P3V.2, CR3.2, D2.A, D3.2, ENCODER_5V.2, LIDAR_12V.2, MOTOR_24V.2, WIFI_5V.2
- net MOTOR_24V_SAFE: now also MOTOR.1; no longer MOTOR_24V.1
- net N$1: now also D1.2, F2.1; no longer D4.2, F3.1
- net N$11: now also LED_3V.A, R2.1; no longer 3VLED.A, R7.1
- net N$14: now also F3.2; no longer F4.2
- net N$18: now also LED_5V.A, R3.1; no longer 5VLED.A, R8.1
- net N$3: now also 24V.1; no longer 24V.2
- net N$6: now also F2.2; no longer F3.2
- net N$8: now also LED_12V.A; no longer 12VLED.A
- net N$9: now also F4.2; no longer F2.2
Routing:
- net 5V: track 0.00 -> 128.3 mm, vias 0 -> 2
- net 24V: track 0.00 -> 103.7 mm
- net GND: track 292.5 -> 395.0 mm, vias 0 -> 3
- net 3.3V: track 0.00 -> 79.2 mm, vias 0 -> 2
- net 24V_SAFE: track 75.9 -> 0.00 mm
- net N$10: track 58.6 -> 0.00 mm
- net 12V: track 0.00 -> 58.0 mm
- net 5V_SAFE: track 53.8 -> 0.00 mm
- net N$12: track 51.1 -> 0.00 mm
- net N$1: track 57.9 -> 17.3 mm
- net N$15: track 0.00 -> 34.1 mm
- net N$4 (its old number): track 27.4 -> 0.00 mm
- net N$9: track 31.9 -> 15.9 mm
- net N$3: track 21.4 -> 8.68 mm
- net N$14: track 23.2 -> 11.3 mm
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
Commit message: Update
Connections:
- net MOTOR_24V_SAFE renamed MOTOR_24V
Changed lines of the file:
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@@
 <wire x1="31.598" y1="16.51" x2="31.598" y2="10.16" width="1.27" layer="1"/>
 </signal>
-<signal name="MOTOR_24V_SAFE" class="6">
+<signal name="MOTOR_24V" class="6">
 <contactref element="MOTOR" pad="1"/>
 <contactref element="F5" pad="2"/>

Commit message: Update
Parts:
- C1: value 10µF -> 1µF
- renumbered 24V to INPUT
Connections:
- removed net N$14: F3.2, U2.3
- removed net N$3 (its old number): F1.1, INPUT.1
- removed net N$6 (its old number): F2.2, U1.3
- removed net N$9: F4.2, U3.3
- new net 12V,PROTECTED: C4.1, D5.C, D6.C, LIDAR.1, R4.2
- new net 24V,PROTECTED: C1.1, CR1.1, CR2.1, F5.1, R1.2, U1.1, U2.1, U3.1
- new net 3.3V,PROTECTED: C2.1, CPU.1, D1.1, D2.1, R2.2
- new net 5V,PROTECTED: C3.1, D3.C, D4.C, ENCODER.1, R3.2, WIFI.1
- net 12V: now also F4.2, U3.3; no longer C4.1, D5.C, D6.C, LIDAR.1, R4.2
- net 24V: now also F1.1, INPUT.1; no longer C1.1, CR1.1, CR2.1, F5.1, R1.2, U1.1, U2.1, U3.1
- net 3.3V: now also F2.2, U1.3; no longer C2.1, CPU.1, D1.1, D2.1, R2.2
- net 5V: now also F3.2, U2.3; no longer C3.1, D3.C, D4.C, ENCODER.1, R3.2, WIFI.1
Routing:
- net 5V,PROTECTED: track 0.00 -> 128.3 mm, vias 0 -> 2
- net 5V: track 128.3 -> 11.3 mm, vias 2 -> 0
- net 24V,PROTECTED: track 0.00 -> 103.7 mm
- net 24V: track 103.7 -> 8.68 mm
- net 3.3V,PROTECTED: track 0.00 -> 79.2 mm, vias 0 -> 2
- net 3.3V: track 79.2 -> 12.0 mm, vias 2 -> 0
- net 12V,PROTECTED: track 0.00 -> 58.0 mm
- net 12V: track 58.0 -> 15.9 mm
- net N$9: track 15.9 -> 0.00 mm
- net N$6 (its old number): track 12.0 -> 0.00 mm
- net N$14: track 11.3 -> 0.00 mm
- net N$3 (its old number): track 8.68 -> 0.00 mm
- net N$2: track 20.2 -> 17.9 mm
Changed lines of the file:
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@@
 </class>
 </classes>
-<designrules name="default">
+<designrules name="default *">
 <description language="de">&lt;b&gt;EAGLE Design Rules&lt;/b&gt;
 &lt;p&gt;
@@
 </autorouter>
 <elements>
-<element name="24V" library="con-molex" package="5566-2" value="5566-2" x="12.7" y="68.58" smashed="yes">
+<element name="INPUT" library="con-molex" package="5566-2" value="5566-2" x="12.7" y="68.58" smashed="yes">
 <attribute name="NAME" x="11.43" y="73.66" size="1.27" layer="25"/>
 <attribute name="VALUE" x="10.16" y="62.23" size="1.27" layer="27"/>
@@
 <attribute name="VALUE" x="21.59" y="7.62" size="1.27" layer="27" rot="R90"/>
 </element>
-<element name="C1" library="rcl" library_urn="urn:adsk.eagle:library:334" package="C1210" package3d_urn="urn:adsk.eagle:package:23619/2" value="10µF" x="22.86" y="25.4" smashed="yes" rot="R180">
+<element name="C1" library="rcl" library_urn="urn:adsk.eagle:library:334" package="C1210" package3d_urn="urn:adsk.eagle:package:23619/2" value="1µF" x="22.86" y="25.4" smashed="yes" rot="R180">
 <attribute name="NAME" x="24.765" y="23.495" size="1.27" layer="25" rot="R180"/>
 <attribute name="POPULARITY" value="6" x="6.35" y="132.08" size="1.778" layer="27" rot="R180" display="off"/>
@@
 <attribute name="POPULARITY" value="6" x="115.57" y="-87.63" size="1.778" layer="27" display="off"/>
 <attribute name="SPICEPREFIX" value="C" x="115.57" y="-87.63" size="1.778" layer="27" display="off"/>
-<attribute name="VALUE" x="81.915" y="15.875" size="1.27" layer="27"/>
+<attribute name="VALUE" x="79.375" y="18.415" size="1.27" layer="27"/>
 </element>
 <element name="CPU" library="con-molex" library_urn="urn:adsk.eagle:library:165" package="70543-02" package3d_urn="urn:adsk.eagle:package:8078681/1" value="C-GRID-02-70543" x="88.9" y="26.67" smashed="yes">
@@
 <attribute name="MANUFACTURER_PART_NUMBER" value="SMAJ26A-E3/61" x="76.2" y="130.81" size="1.778" layer="27" rot="R90" display="off"/>
 <attribute name="MFR_NAME" value="Vishay" x="76.2" y="130.81" size="1.778" layer="27" rot="R90" display="off"/>
-<attribute name="NAME" x="24.765" y="64.0334" size="1.27" layer="27" ratio="6" rot="SR90"/>
-<attribute name="VALUE" x="24.765" y="65.5828" size="1.27" layer="21" ratio="6" rot="SR90"/>
+<attribute name="NAME" x="22.225" y="60.2234" size="1.27" layer="27" ratio="6" rot="SR0"/>
+<attribute name="VALUE" x="20.955" y="61.7728" size="1.27" layer="21" ratio="6" rot="SR0"/>
 </element>
 <element name="CR2" library="SMAJ26A-E361" package="DIODE_DO-214AC" value="SMAJ26A-E3/61" x="33.02" y="53.34" smashed="yes" rot="R180">
@@
 <attribute name="MANUFACTURER_PART_NUMBER" value="SMAJ26A-E3/61" x="5.08" y="143.51" size="1.778" layer="27" rot="R180" display="off"/>
 <attribute name="MFR_NAME" value="Vishay" x="5.08" y="143.51" size="1.778" layer="27" rot="R180" display="off"/>
-<attribute name="NAME" x="36.2966" y="53.975" size="1.27" layer="27" ratio="6" rot="SR180"/>
-<attribute name="VALUE" x="34.7472" y="53.975" size="1.27" layer="21" ratio="6" rot="SR180"/>
+<attribute name="NAME" x="24.8666" y="51.435" size="1.27" layer="27" ratio="6" rot="SR0"/>
+<attribute name="VALUE" x="22.0472" y="55.245" size="1.27" layer="21" ratio="6" rot="SR0"/>
 </element>
 <element name="D1" library="SMBJ3V3-E352" package="VISHAY_SMBJ3V3-E3-52_0" value="VISHAY_SMBJ3V3-E3-52VISHAY_SMBJ3V3-E3-52_0_0" x="78.74" y="31.75" smashed="yes" rot="R90">
@@
 <attribute name="MF" value="" x="-19.05" y="-55.88" size="1.778" layer="27" rot="R270" display="off"/>
 <attribute name="MPN" value="" x="-19.05" y="-55.88" size="1.778" layer="27" rot="R270" display="off"/>
-<attribute name="NAME" x="64.77" y="33.401" size="1.27" layer="25" ratio="10" rot="R270"/>
+<attribute name="NAME" x="64.77" y="28.321" size="1.27" layer="25" ratio="10" rot="R270"/>
 <attribute name="OC_FARNELL" value="unknown" x="-19.05" y="-55.88" size="1.778" layer="27" rot="R270" display="off"/>
 <attribute name="OC_NEWARK" value="unknown" x="-19.05" y="-55.88" size="1.778" layer="27" rot="R270" display="off"/>
 <attribute name="POPULARITY" value="0" x="-19.05" y="-55.88" size="1.778" layer="27" rot="R270" display="off"/>
-<attribute name="VALUE" x="58.42" y="33.528" size="1.27" layer="27" ratio="10" rot="R270"/>
+<attribute name="VALUE" x="58.42" y="28.448" size="1.27" layer="27" ratio="10" rot="R270"/>
 </element>
 <element name="F3" library="fuse" library_urn="urn:adsk.eagle:library:233" package="TE5" package3d_urn="urn:adsk.eagle:package:14069/1" value="1.5A" x="35.56" y="39.37" smashed="yes" rot="R180">
@@
 <attribute name="MANUFACTURER_PART_NUMBER" value="MIC29300-3.3WU" x="80.01" y="7.62" size="1.778" layer="27" display="off"/>
 <attribute name="MFR_NAME" value="Micrel" x="80.01" y="7.62" size="1.778" layer="27" display="off"/>
-<attribute name="NAME" x="44.9834" y="33.655" size="1.27" layer="27" ratio="6" rot="SR0"/>
-<attribute name="VALUE" x="46.5328" y="33.655" size="1.27" layer="21" ratio="6" rot="SR0"/>
+<attribute name="NAME" x="43.7134" y="31.115" size="1.27" layer="27" ratio="6" rot="SR0"/>
+<attribute name="VALUE" x="42.7228" y="29.845" size="1.27" layer="21" ratio="6" rot="SR0"/>
 </element>
 <element name="U2" library="MIC29300-5.0WU" package="TO-263-3_MCL" value="MIC29300-5.0WU" x="12.7" y="36.83" smashed="yes" rot="R90">
@@
 <contactref element="CR2" pad="2"/>
 <contactref element="C1" pad="2"/>
-<contactref element="24V" pad="2"/>
+<contactref element="INPUT" pad="2"/>
 <wire x1="14.122" y1="10.16" x2="17.78" y2="6.502" width="1.27" layer="1"/>
 <wire x1="17.78" y1="6.502" x2="17.78" y2="6.35" width="1.27" layer="1"/>
@@
 <via x="25.4" y="36.83" extent="1-16" drill="0.35"/>
 </signal>
-<signal name="N$9">
+<signal name="12V">
 <contactref element="F4" pad="2"/>
 <contactref element="U3" pad="3"/>
@@
 <wire x1="45.72" y1="59.5249" x2="45.72" y2="50.8" width="1.27" layer="1"/>
 </signal>
-<signal name="N$6">
+<signal name="3.3V">
 <contactref element="F2" pad="2"/>
 <contactref element="U1" pad="3"/>
@@
 <wire x1="60.7949" y1="25.2349" x2="62.23" y2="26.67" width="1.27" layer="1"/>
 </signal>
-<signal name="5V" class="2">
+<signal name="5V,PROTECTED" class="2">
 <contactref element="ENCODER" pad="1"/>
 <contactref element="D3" pad="C"/>
@@
 <wire x1="35.56" y1="34.29" x2="55.88" y2="34.29" width="1.27" layer="16"/>
 </signal>
-<signal name="N$14">
+<signal name="5V">
 <contactref element="F3" pad="2"/>
 <contactref element="U2" pad="3"/>
 <wire x1="21.7551" y1="39.37" x2="33.02" y2="39.37" width="1.27" layer="1"/>
 </signal>
-<signal name="24V" class="3">
+<signal name="24V,PROTECTED" class="3">
 <contactref element="F5" pad="1"/>
 <contactref element="U1" pad="1"/>
@@
 <contactref element="F1" pad="2"/>
 <contactref element="CR1" pad="2"/>
-<wire x1="24.13" y1="69.0118" x2="24.13" y2="71.12" width="1.27" layer="1"/>
-<wire x1="24.13" y1="71.12" x2="21.59" y2="71.12" width="1.27" layer="1"/>
-<wire x1="21.59" y1="71.12" x2="20.551" y2="70.081" width="1.27" layer="1"/>
-<wire x1="20.551" y1="70.081" x2="20.551" y2="69.5648125" width="1.27" layer="1"/>
-<wire x1="20.551" y1="69.5648125" x2="17.78" y2="66.7938125" width="1.27" layer="1"/>
-<wire x1="17.78" y1="66.7938125" x2="17.78" y2="57.15" width="1.27" layer="1"/>
+<wire x1="24.13" y1="69.0118" x2="23.2918" y2="69.85" width="1.27" layer="1"/>
+<wire x1="23.2918" y1="69.85" x2="20.32" y2="69.85" width="1.27" layer="1"/>
+<wire x1="20.32" y1="69.85" x2="17.78" y2="67.31" width="1.27" layer="1"/>
+<wire x1="17.78" y1="67.31" x2="17.78" y2="57.15" width="1.27" layer="1"/>
 </signal>
 <signal name="N$5">
@@
 <wire x1="57.15" y1="29.21" x2="70.695" y2="29.21" width="1.27" layer="1"/>
 </signal>
-<signal name="N$8">
+<signal name="N$3">
 <contactref element="R4" pad="1"/>
 <contactref element="LED_12V" pad="A"/>
@@
 <wire x1="69.85" y1="31.75" x2="71.689" y2="33.589" width="1.27" layer="1"/>
 </signal>
-<signal name="N$11">
+<signal name="N$6">
 <contactref element="R2" pad="1"/>
 <contactref element="LED_3V" pad="A"/>
@@
 <wire x1="73.66" y1="54.61" x2="48.26" y2="54.61" width="1.27" layer="1"/>
 </signal>
-<signal name="N$15">
+<signal name="N$8">
 <contactref element="F3" pad="1"/>
 <contactref element="D3" pad="A"/>
@@
 <wire x1="50.8" y1="50.8" x2="65.195" y2="50.8" width="1.27" layer="1"/>
 </signal>
-<signal name="12V" class="4">
+<signal name="12V,PROTECTED" class="4">
 <contactref element="LIDAR" pad="1"/>
 <contactref element="D5" pad="C"/>
@@
 <wire x1="77.47" y1="14.1" x2="77.47" y2="13.545" width="1.27" layer="1"/>
 </signal>
-<signal name="3.3V">
+<signal name="3.3V,PROTECTED">
 <contactref element="D1" pad="1"/>
 <contactref element="CPU" pad="1"/>
@@
 <via x="74.93" y="29.21" extent="1-16" drill="0.35"/>
 </signal>
-<signal name="N$18">
+<signal name="N$7">
 <contactref element="LED_5V" pad="A"/>
 <contactref element="R3" pad="1"/>
 <wire x1="11.278" y1="16.51" x2="11.278" y2="10.16" width="1.27" layer="1"/>
 </signal>
-<signal name="N$3">
-<contactref element="24V" pad="1"/>
+<signal name="24V">
+<contactref element="INPUT" pad="1"/>
 <contactref element="F1" pad="1"/>
 <wire x1="12.7" y1="65.83" x2="12.7" y2="57.15" width="1.27" layer="1"/>
@@
 <mfgpreviewcolor name="substratecolor" color="0xFF786E46"/>
 </mfgpreviewcolors>
-<errors>
-</errors>
 </board>
 </drawing>

Commit message: Update
Parts:
- C1: value 1µF -> 40µF
- C2, C3: value 1µF -> 10µF
- C4: value 1µF -> 20µF
- turned CR1 to 180 degrees
Routing:
- net N$2: track 17.9 -> 12.1 mm
- net 24V,PROTECTED: track 103.7 -> 100.2 mm
- net GND: track 395.0 -> 397.3 mm
