File: TeamG_PCB.sch (EAGLE design)
At the start: 34 parts, among them U1 MIC29300-3.3WU, U2 MIC29300-5.0WU, U3 MIC29300-12WU

Commit message: Update
Parts:
- removed 12VLED: 0, led:LEDSMT1206
- removed C6: 1µF, rcl:C-USC1210
- removed CR3: SMAJ26A-E3/61, SMAJ26A-E361:SMAJ26A-E3/61
- removed LIDAR_12V, MOTOR_24V: C-GRID-02-70543, con-molex:C-GRID-02-70543
- added C4: 1µF, rcl:C-USC1210
- added CR2: SMAJ26A-E3/61, SMAJ26A-E361:SMAJ26A-E3/61
- added LED_12V: 0, led:LEDSMT1206
- added LIDAR, MOTOR: C-GRID-02-70543, con-molex:C-GRID-02-70543
- D1, D2: value P4SMA16A -> VISHAY_SMBJ3V3-E3-52VISHAY_SMBJ3V3-E3-52_0_0; device P4SMA16A:P4SMA16A -> SMBJ3V3-E352:VISHAY_SMBJ3V3-E3-52VISHAY_SMBJ3V3-E3-52_0_0
- D3, D4: value VISHAY_SMBJ3V3-E3-52VISHAY_SMBJ3V3-E3-52_0_0 -> SMAJ5.0; device SMBJ3V3-E352:VISHAY_SMBJ3V3-E3-52VISHAY_SMBJ3V3-E3-52_0_0 -> SMAJ5.0:SMAJ5.0
- D5, D6: value SMAJ5.0 -> P4SMA16A; device SMAJ5.0:SMAJ5.0 -> P4SMA16A:P4SMA16A
- F2: value 3A -> 1.5A
- F4: value 1.5A -> 3A
- R1: value 1100Ω -> 1000Ω
- R2: value 65Ω -> 100Ω
- renumbered 3VLED to LED_3V, 5VLED to LED_5V, CPU_3P3V to CPU, ENCODER_5V to ENCODER, R7 to R2, R8 to R3, WIFI_5V to WIFI
Connections:
- removed net 24V_SAFE: C1.1, CR1.1, CR3.1, F5.1, R1.2, U1.IN, U2.IN, U3.IN
- removed net 5V_SAFE: C3.1, D5.C, D6.C, ENCODER-1.S, R3.2, WIFI-1.S
- removed net N$10: C2.1, CPU-1.S, D3.CATHODE, D4.CATHODE, R2.2
- removed net N$12: C6.1, D1.C, D2.C, LIDAR_12V-1.S, R4.2
- removed net N$4 (its old number): D1.A, F2.1
- new net 12V: C4.1, D5.C, D6.C, LIDAR-1.S, R4.2
- new net 24V: C1.1, CR1.1, CR2.1, F5.1, R1.2, U1.IN, U2.IN, U3.IN
- new net 3.3V: C2.1, CPU-1.S, D1.CATHODE, D2.CATHODE, R2.2
- new net 5V: C3.1, D3.C, D4.C, ENCODER-1.S, R3.2, WIFI-1.S
- new net N$15: D3.A, F3.1
- net GND: now also 24V-2.S, C4.2, CR2.2, D2.ANODE, D4.A, LED_12V.C, LIDAR-2.S, MOTOR-2.S; no longer 12VLED.C, 24V-1.S, C6.2, CR3.2, D2.A, D3.ANODE, LIDAR_12V-2.S, MOTOR_24V-2.S
- net MOTOR_24V_SAFE: now also MOTOR-1.S; no longer MOTOR_24V-1.S
- net N$1: now also D1.ANODE, F2.1; no longer D4.ANODE, F3.1
- net N$14: now also F3.2; no longer F4.2
- net N$3: now also 24V-1.S; no longer 24V-2.S
- net N$6: now also F2.2; no longer F3.2
- net N$8: now also LED_12V.A; no longer 12VLED.A
- net N$9: now also F4.2; no longer F2.2
Other:
- moved on the sheet: 24V-1, 24V-2, C1, CR1, D5, D6, F1, F2, F3, F4, F5, R1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

Commit message: Update
Connections:
- net MOTOR_24V_SAFE renamed MOTOR_24V
Changed lines of the file:
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@@
 </segment>
 </net>
-<net name="MOTOR_24V_SAFE" class="6">
+<net name="MOTOR_24V" class="6">
 <segment>
 <pinref part="MOTOR" gate="-1" pin="S"/>

Commit message: Update
Parts:
- removed 24V: 5566-2, con-molex:5566-2
- added INPUT: 5566-2, con-molex:5566-2
- C1: value 10µF -> 1µF
Connections:
- removed net N$14: F3.2, U2.OUT
- removed net N$3 (its old number): 24V-1.S, F1.1
- removed net N$6 (its old number): F2.2, U1.OUT
- removed net N$9: F4.2, U3.OUT
- new net 12V,PROTECTED: C4.1, D5.C, D6.C, LIDAR-1.S, R4.2
- new net 24V,PROTECTED: C1.1, CR1.1, CR2.1, F5.1, R1.2, U1.IN, U2.IN, U3.IN
- new net 3.3V,PROTECTED: C2.1, CPU-1.S, D1.CATHODE, D2.CATHODE, R2.2
- new net 5V,PROTECTED: C3.1, D3.C, D4.C, ENCODER-1.S, R3.2, WIFI-1.S
- net 12V: now also F4.2, U3.OUT; no longer C4.1, D5.C, D6.C, LIDAR-1.S, R4.2
- net 24V: now also F1.1, INPUT-1.S; no longer C1.1, CR1.1, CR2.1, F5.1, R1.2, U1.IN, U2.IN, U3.IN
- net 3.3V: now also F2.2, U1.OUT; no longer C2.1, CPU-1.S, D1.CATHODE, D2.CATHODE, R2.2
- net 5V: now also F3.2, U2.OUT; no longer C3.1, D3.C, D4.C, ENCODER-1.S, R3.2, WIFI-1.S
- net GND: now also INPUT-2.S; no longer 24V-2.S
Other:
- moved on the sheet: C1, C2, C3, C4, CPU-1, CPU-2, CR1, CR2, D1, D2, D3, D4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

Commit message: Update
Parts:
- C1: value 1µF -> 40µF
- C2, C3: value 1µF -> 10µF
- C4: value 1µF -> 20µF
Changed lines of the file:
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@@
 <parts>
 <part name="F1" library="fuse" library_urn="urn:adsk.eagle:library:233" deviceset="TE5" device="" package3d_urn="urn:adsk.eagle:package:14069/1" value="21A"/>
-<part name="C1" library="rcl" library_urn="urn:adsk.eagle:library:334" deviceset="C-US" device="C1210" package3d_urn="urn:adsk.eagle:package:23619/2" value="1µF"/>
+<part name="C1" library="rcl" library_urn="urn:adsk.eagle:library:334" deviceset="C-US" device="C1210" package3d_urn="urn:adsk.eagle:package:23619/2" value="40µF"/>
 <part name="R1" library="rcl" library_urn="urn:adsk.eagle:library:334" deviceset="R-US_" device="R1206" package3d_urn="urn:adsk.eagle:package:23540/2" value="1000Ω"/>
 <part name="24VLED" library="led" library_urn="urn:adsk.eagle:library:259" deviceset="LED" device="SMT1206" package3d_urn="urn:adsk.eagle:package:15796/2" value="0"/>
@@
 <part name="GND4" library="supply1" library_urn="urn:adsk.eagle:library:371" deviceset="GND" device=""/>
 <part name="F4" library="fuse" library_urn="urn:adsk.eagle:library:233" deviceset="TE5" device="" package3d_urn="urn:adsk.eagle:package:14069/1" value="3A"/>
-<part name="C4" library="rcl" library_urn="urn:adsk.eagle:library:334" deviceset="C-US" device="C1210" package3d_urn="urn:adsk.eagle:package:23619/2" value="1µF"/>
+<part name="C4" library="rcl" library_urn="urn:adsk.eagle:library:334" deviceset="C-US" device="C1210" package3d_urn="urn:adsk.eagle:package:23619/2" value="20µF"/>
 <part name="R4" library="rcl" library_urn="urn:adsk.eagle:library:334" deviceset="R-US_" device="R1206" package3d_urn="urn:adsk.eagle:package:23540/2" value="500Ω"/>
 <part name="LED_12V" library="led" library_urn="urn:adsk.eagle:library:259" deviceset="LED" device="SMT1206" package3d_urn="urn:adsk.eagle:package:15796/2" value="0"/>
@@
 <part name="D4" library="SMAJ5.0" deviceset="SMAJ5.0" device=""/>
 <part name="F5" library="fuse" library_urn="urn:adsk.eagle:library:233" deviceset="TE5" device="" package3d_urn="urn:adsk.eagle:package:14069/1" value="15A"/>
-<part name="C2" library="rcl" library_urn="urn:adsk.eagle:library:334" deviceset="C-US" device="C1210" package3d_urn="urn:adsk.eagle:package:23619/2" value="1µF"/>
-<part name="C3" library="rcl" library_urn="urn:adsk.eagle:library:334" deviceset="C-US" device="C1210" package3d_urn="urn:adsk.eagle:package:23619/2" value="1µF"/>
+<part name="C2" library="rcl" library_urn="urn:adsk.eagle:library:334" deviceset="C-US" device="C1210" package3d_urn="urn:adsk.eagle:package:23619/2" value="10µF"/>
+<part name="C3" library="rcl" library_urn="urn:adsk.eagle:library:334" deviceset="C-US" device="C1210" package3d_urn="urn:adsk.eagle:package:23619/2" value="10µF"/>
 <part name="GND5" library="supply1" library_urn="urn:adsk.eagle:library:371" deviceset="GND" device=""/>
 <part name="GND6" library="supply1" library_urn="urn:adsk.eagle:library:371" deviceset="GND" device=""/>
